Commit message: Added launch option to use real or simulated controllers; added camera hitbox to urdf

File: ur_e_description/urdf/ur5e.urdf.xacro (robot description, xacro)
@@ -49,5 +49,6 @@
     <xacro:property name="wrist_radius" value="0.045" />      <!-- manually measured -->
     <!-- This is for compatibility reasons, as transformation between base and base_link was always 180 degree in the ur_description -->
-    <xacro:property name="base_correction" value="${pi}" />
+    <!-- Actually, do not need to do base correction, so set to 0 -->
+    <xacro:property name="base_correction" value="0" />
     <link name="${prefix}base_link" >
       <visual>
@@ -309,10 +310,20 @@
       <origin xyz="0.0 0.0 0.0" rpy="0.0 ${-pi/2.0} ${pi/2.0}" />
     </joint>
+    <!-- Camera on the end effector -->
     <link name="${prefix}ee_link">
-      <collision>
-        <geometry>
-          <box size="0.01 0.01 0.01"/>
-        </geometry>
-        <origin rpy="0 0 0" xyz="-0.01 0 0"/>
+      <visual>
+        <geometry>
+          <box size="0.09 0.1 0.18"/>
+        </geometry>
+        <origin rpy="0.7854 0 0" xyz="0.045 0 0"/> <!-- Note that axes are different to the ones shown on the UR5e tablet -->
+        <material name="LightGrey">
+          <color rgba="0.7 0.7 0.7 1.0"/>
+        </material>
+      </visual>
+      <collision>
+        <geometry>
+          <box size="0.09 0.1 0.18"/> <!-- Changed for camera - default 0.01 0.01 0.01 -->
+        </geometry>
+        <origin rpy="0.7854 0 0" xyz="0.045 0 0"/>
       </collision>
     </link>
